Commit message: 抓取规划与控制开发

File: src/openarm_description/urdf/robot/v10.urdf.xacro (robot description, xacro)
@@ -70,5 +70,5 @@
       <geometry>
         <!-- Use D435 mesh from openarm_mujoco (under v1/meshes/visual/cam) -->
-        <mesh filename="file:///home/zjc/openarm_ws/openarm_mujoco/v1/meshes/visual/cam/d435_0.stl"/>
+        <mesh filename="file:///home/chenwei/openarm_ws/openarm_mujoco/v1/meshes/visual/cam/d435_0.stl"/>
       </geometry>
       <material name="d435_material">
@@ -127,5 +127,5 @@
       <geometry>
         <!-- Absolute path to banana mesh in openarm_mujoco -->
-        <mesh filename="file:///home/zjc/openarm_ws/openarm_mujoco/v1/meshes/011_banana/textured_simple.obj"/>
+        <mesh filename="file:///home/chenwei/openarm_ws/openarm_mujoco/v1/meshes/011_banana/textured_simple.obj"/>
       </geometry>
     </visual>

Commit message: 修改路径参数，机械臂移动速度，语法错误，运行起来，机械抓移动到错误位置

File: src/openarm_description/urdf/robot/v10.urdf.xacro (robot description, xacro)
@@ -67,5 +67,5 @@
       <origin xyz="0.04 0.0 0.62" rpy="3.14 1.3 0"/>
       <geometry>
-        <mesh filename="file:///home/ros/openarm_ws/openarm_mujoco/v1/meshes/visual/cam/d435_0.stl"/>
+        <mesh filename="file:///home/zjc/openarm_ws/openarm_mujoco/v1/meshes/visual/cam/d435_0.stl"/>
       </geometry>
       <material name="d435_material">
@@ -116,5 +116,5 @@
       <origin xyz="0.35 0 0.35" rpy="0 0 1.57"/>
       <geometry>
-        <mesh filename="file:///home/chenwei/openarm_ws/openarm_mujoco/v1/meshes/011_banana/textured_simple.obj"/>
+        <mesh filename="file:///home/zcj/openarm_ws/openarm_mujoco/v1/meshes/011_banana/textured_simple.obj"/>
       </geometry>
     </visual>
